File: D-SUB-Tester.kicad_pcb (KiCad board)
At the start: 2 copper layers, 180 x 130.5 mm, 54 parts, among them J1 DE9_Plug_MountingHoles, J2 DE9_Receptacle_MountingHoles, J3 DE9_Plug_MountingHoles, J4 DE9_Receptacle_MountingHoles, J5 Unbetitelte Telefunken-Anzeig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, J6 USB_C_Receptacle_PowerOnly_6P, J7 ICSP, SW1 SW_Reed_SPDT, SW2 SW_Reed_SPDT, SW3 SW_Reed_SPDT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

Commit message: quick save
Other:
- board text added: ">"
- board text added: "A"
- board text added: "B"

Commit message: EVT 1
Parts:
- added REF**: MountingHole_3.2mm_M3, MountingHole:MountingHole_3.2mm_M3, F.Cu at (174.0, 80.0)
- added REF**: MountingHole_3.2mm_M3, MountingHole:MountingHole_3.2mm_M3, F.Cu at (174.0, 152.0)
- added REF**: MountingHole_3.2mm_M3, MountingHole:MountingHole_3.2mm_M3, F.Cu at (30.0, 152.0)
- added REF**: MountingHole_3.2mm_M3, MountingHole:MountingHole_3.2mm_M3, F.Cu at (174.0, 118.0)
- added REF**: MountingHole_3.2mm_M3, MountingHole:MountingHole_3.2mm_M3, F.Cu at (143.0, 152.0)
- added REF**: MountingHole_3.2mm_M3, MountingHole:MountingHole_3.2mm_M3, F.Cu at (30.0, 80.0)
- added REF**: MountingHole_3.2mm_M3, MountingHole:MountingHole_3.2mm_M3, F.Cu at (87.0, 80.0)
- moved SW1 99.8 mm to (128.0, 32.2), turned to 90 degrees
- moved R11 55.8 mm to (154.7, 29.0), turned to 180 degrees
- moved D2 45.3 mm to (110.0, 152.3)
- moved D4 40.4 mm to (105.0, 152.3)
- moved D6 35.5 mm to (100.0, 152.3)
- moved D8 30.7 mm to (95.0, 152.3)
- moved SW2 26.0 mm to (128.0, 42.8)
- moved SW3 26.0 mm to (128.0, 53.1)
- moved SW4 26.0 mm to (128.0, 63.6)
- moved R1 25.9 mm to (106.2, 93.2)
- moved R15 25.9 mm to (122.7, 100.4)
- moved R5 25.9 mm to (127.7, 97.7)
- moved C1 25.9 mm to (188.5, 49.0)
- moved C2 25.9 mm to (118.5, 83.0)
- moved C3 25.9 mm to (54.0, 90.5)
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Routing:
- net Net-(D2-A): track 64.3 -> 88.4 mm, vias 0 -> 2
- net Net-(D4-A): track 76.6 -> 97.8 mm, vias 0 -> 2
- net Net-(D6-A): track 87.2 -> 105.9 mm, vias 0 -> 2
- net Net-(U1-AN1/RA1): track 8.56 -> 27.2 mm, vias 0 -> 2
- net Net-(D8-A): track 99.4 -> 115.4 mm, vias 0 -> 2
- net Net-(U1-CLKIN/OSC1/RA7): track 166.0 -> 153.9 mm
- net Net-(D9-A): track 103.9 -> 93.3 mm
- net Net-(R14-Pad2): track 16.5 -> 24.3 mm
- net VDD: track 351.8 -> 344.2 mm
- net Net-(R11-Pad2): track 3.93 -> 11.1 mm
- net Net-(R13-Pad2): track 12.1 -> 18.8 mm
- net Net-(D7-A): track 90.4 -> 84.2 mm
- net Net-(D5-A): track 78.8 -> 74.7 mm
- net Net-(R12-Pad2): track 10.1 -> 13.3 mm
- net GND: track 13.9 -> 16.6 mm
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Other:
- board size 180 x 130.5 mm -> 177 x 134 mm
- board text added: "9 8 7 6 5 4 3 2 1"
- board text added: "PROGRAMM"
- board text removed: "AKTUELLES PROGRAMM"
- board text removed: "todo: mounting holes, beschriftung, constrains"
